File: KiCAD/ADC.kicad_sch (KiCad schematic)
At the start: 25 parts, among them IC1 AK5572EN, U5 74LVC1G80

Commit message: 初步layout
Parts:
- removed CE2: 220u 10V, symbol Device:C_Polarized_Small
- removed R26, R27, R28, R29: 4.7k, symbol Device:R_Small
- removed R34: 100, symbol Device:R_Small
- added C18, C20, C21, C23: 100p, Capacitor_SMD:C_0402_1005Metric, symbol Device:C_Small
- added C19, C22: 15n, Capacitor_SMD:C_0402_1005Metric, symbol Device:C_Small
- added R22, R23, R24, R25: 10, Resistor_SMD:R_0402_1005Metric, symbol Device:R_Small
- C24: renamed from C16; footprint (none) -> Capacitor_SMD:C_0402_1005Metric
- C25: renamed from C17; footprint (none) -> Capacitor_SMD:C_0402_1005Metric
- C26: renamed from C18; footprint (none) -> Capacitor_SMD:C_0402_1005Metric
- C27: renamed from C19; footprint (none) -> Capacitor_SMD:C_0402_1005Metric
- C28: renamed from C20; footprint (none) -> Capacitor_SMD:C_0603_1608Metric
- C29: renamed from C21; footprint (none) -> Capacitor_SMD:C_0603_1608Metric
- C30: renamed from C22; footprint (none) -> Capacitor_SMD:C_0603_1608Metric
- C31: renamed from C23; footprint (none) -> Capacitor_SMD:C_0402_1005Metric
- C32: renamed from C24; footprint (none) -> Capacitor_SMD:C_0402_1005Metric
- CE1: footprint (none) -> Capacitor_Tantalum_SMD:CP_EIA-3528-21_Kemet-B
- IC1: footprint QFN48_7x7-0p5_AKM -> Package_DFN_QFN:QFN-48-1EP_7x7mm_P0.5mm_EP5.1x5.1mm_ThermalVias
- R30, R31, R32: footprint (none) -> Resistor_SMD:R_0402_1005Metric
- R33: footprint (none) -> Resistor_SMD:R_0805_2012Metric
- R34: renamed from R35; footprint (none) -> Resistor_SMD:R_0402_1005Metric
- R35: renamed from R36; value 22 -> 100; footprint (none) -> Resistor_SMD:R_0402_1005Metric
- U7: renamed from U5; footprint (none) -> Package_TO_SOT_SMD:SOT-353_SC-70-5
- Y1: value (none) -> NZ2520SDA; footprint (none) -> Oscillator:Oscillator_SMD_SeikoEpson_SG210-4Pin_2.5x2.0mm
Connections:
- net +3.3VD: no longer C26.1, C29.1, IC1.17 (TVDD)
- net GND: now also IC1.41 (PSN/CAD0_SPI), C18.1, C20.2, C21.1, C23.2
- net IN1_N: now also C19.2, C20.1, R23.1; no longer IC1.48 (AIN1N)
- net IN1_P: now also C18.2, C19.1, R22.1; no longer IC1.47 (AIN1P)
- net IN2_N: now also C21.2, C22.1, R24.1; no longer IC1.4 (AIN2N)
- net IN2_P: now also C22.2, C23.1, R25.1; no longer IC1.5 (AIN2P)
- net at IC1.25 (BICK/DCLK), R30.1: now also U7.2 (C)
- net TVDD: now reaches IC1.24 (MSN)
- net TVDD: now also C26.1, C29.1, IC1.17 (TVDD), IC1.42 (I2C), IC1.45 (LDOE)
- new net: IC1.48 (AIN1N), R23.2
- new net: IC1.47 (AIN1P), R22.2
- new net: IC1.4 (AIN2N), R24.2
- new net: IC1.5 (AIN2P), R25.2
Other:
- moved on the sheet: C24, C25, C26, C27, C28, C29, C30, CE1, IC1, R30, R31, R32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
