File: KiCAD/AFE.kicad_sch (KiCad schematic)
At the start: 37 parts, among them U2 OPA1656ID, U3 THS4551xRGT, U4 THS4551xRGT

Commit message: 初步layout
Parts:
- removed C8: 100p, symbol Device:C_Small
- removed C9: 15n, symbol Device:C_Small
- removed R22, R23, R24, R25: 10, symbol Device:R_Small
- removed U2: OPA1656ID, Package_SO:SOIC-8_3.9x4.9mm_P1.27mm, symbol Amplifier_Operational:OPA1656ID
- removed unit 1 of U3
- added C14, C15: 100p, Capacitor_SMD:C_0402_1005Metric, symbol Device:C_Small
- added C6, C7: 1u, Capacitor_SMD:C_0402_1005Metric, symbol Device:C_Small
- added U3: OPA1655D, Package_SO:SOIC-8_3.9x4.9mm_P1.27mm, symbol Amplifier_Operational:OPA1655D
- added U4: OPA1655DBV, Package_TO_SOT_SMD:SOT-23-5, symbol Amplifier_Operational:OPA1655DBV
- added unit 1 of U5
- C10, C11: value 100p -> 1n; footprint (none) -> Capacitor_SMD:C_0402_1005Metric
- C12: value 15n -> 100p; footprint (none) -> Capacitor_SMD:C_0402_1005Metric
- C13, C3, C5: footprint (none) -> Capacitor_SMD:C_0402_1005Metric
- C16: renamed from C14; footprint (none) -> Capacitor_SMD:C_0402_1005Metric
- C17: renamed from C15; footprint (none) -> Capacitor_SMD:C_0402_1005Metric
- C4: footprint (none) -> Capacitor_SMD:C_0805_2012Metric
- C8: renamed from C6; footprint (none) -> Capacitor_SMD:C_0402_1005Metric
- C9: renamed from C7; footprint (none) -> Capacitor_SMD:C_0402_1005Metric
- MK1: footprint (none) -> Connector_Wire:SolderWire-0.5sqmm_1x02_P4.6mm_D0.9mm_OD2.1mm
- R10, R11, R12, R13, R14, R15, R16, R17, R18, R19, R20, R21, R7, R8: footprint (none) -> Resistor_SMD:R_0402_1005Metric
- R6, R9: footprint (none) -> Resistor_SMD:R_0805_2012Metric
- renumbered U3 to U5, U4 to U6
Connections:
- net +2.56V: now also U4.1, U4.4 (-), U5.9 (VOCM)
- net +5VA: now also U5.12 (~{PD})
- net +7V: now also C6.1, U3.7 (V+), U4.5 (V+)
- net -5V: now also C7.1, U3.4 (V-); no longer C9.1
- net GND: now also R10.1, C6.2, C7.2; no longer C10.2, C11.1, C13.2, R11.1
- net OUT1_N: now also R19.2
- net OUT1_P: now also R18.2
- net OUT2_N: now also R20.2
- net OUT2_P: now also R21.2
- net at R20.1: now also U6.11 (OUT-); no longer U6.10 (OUT+)
- net at R14.2: now also C12.2, U5.1 (FB-)
- net at R18.1: now also U5.11 (OUT-)
- net at R19.1: now also U5.10 (OUT+)
- net at R10.2, R14.1: now also C10.1, C12.1, U5.2 (IN+)
- net at R11.2, R15.1: now also C10.2, C13.1, U5.3 (IN-)
- net at R15.2: now also C13.2, U5.4 (FB+)
- net at C4.2, R9.1: now also U3.3 (+)
- net at C5.1, R7.2, R8.1: now also U4.3 (+)
- net at R13.2, R17.1, U6.3 (IN-): now also C11.2, C15.1
- net at R12.1: now also R11.1, U3.2 (-), U3.6; no longer R10.1
- net at R12.2, R16.1, U6.2 (IN+): now also C11.1, C14.1
- net at R16.2, U6.1 (FB-): now also C14.2
- net at R21.1: now also U6.10 (OUT+); no longer U6.11 (OUT-)
- net at R17.2, U6.4 (FB+): now also C15.2
- new net 0: C9.1, U4.2 (V-)
Other:
- note removed: "VOUT≈9Vpp"
- moved on the sheet: C8, C9, R10, R11, R12, R13
