File: KiCAD/MCU.kicad_sch (KiCad schematic)
At the start: 12 parts, among them U6 STM32L432KCUx

Commit message: 初步layout
Parts:
- removed R40, R41: 22, symbol Device:R_Small
- added TP1: SWCLK, TestPoint:TestPoint_Pad_D1.0mm, symbol Connector:TestPoint
- added TP2: SWDIO, TestPoint:TestPoint_Pad_D1.0mm, symbol Connector:TestPoint
- C33: renamed from C25; footprint (none) -> Capacitor_SMD:C_0402_1005Metric
- C34: renamed from C26; footprint (none) -> Capacitor_SMD:C_0603_1608Metric
- C35: renamed from C27; footprint (none) -> Capacitor_SMD:C_0402_1005Metric
- C36: renamed from C28; footprint (none) -> Capacitor_SMD:C_0402_1005Metric
- C37: renamed from C29; footprint (none) -> Capacitor_SMD:C_0402_1005Metric
- JP1: footprint (none) -> Jumper:SolderJumper-2_P1.3mm_Open_RoundedPad1.0x1.5mm
- R36: renamed from R37; footprint (none) -> Resistor_SMD:R_0402_1005Metric
- R37: renamed from R38; footprint (none) -> Resistor_SMD:R_0402_1005Metric
- R38: renamed from R39; footprint (none) -> Resistor_SMD:R_0402_1005Metric
- U8: renamed from U6; footprint Package_DFN_QFN:QFN-32-1EP_5x5mm_P0.5mm_EP3.45x3.45mm -> Package_DFN_QFN:QFN-32-1EP_5x5mm_P0.5mm_EP3.45x3.45mm_ThermalVias
Connections:
- net D+: now also U8.22 (PA12)
- net D-: now also U8.21 (PA11)
- net at U8.23 (PA13): now also TP2.1
- net at U8.24 (PA14): now also TP1.1
- no-connect marks 16 -> 14
