File: KiCAD/Microphone.kicad_sch (KiCad schematic)
At the start: 11 parts, among them J1 USB_C_Receptacle_USB2.0_14P, U1 TPS25200DRVR

Commit message: 初步layout
Parts:
- removed D1: ESD5Zxx, Diode_SMD:D_SOD-523, symbol Diode:ESD5Zxx
- added U1: PRTR5V0U2F, Package_TO_SOT_SMD:SOT-886, symbol Power_Protection:USBLC6-2P6
- C1: value 100n 1kV -> 1n 1kV; footprint (none) -> Capacitor_SMD:C_1206_3216Metric
- C2: footprint (none) -> Capacitor_SMD:C_0402_1005Metric
- H1: footprint (none) -> MountingHole:MountingHole_2.2mm_M2_Pad_Via
- J1: footprint (none) -> Connector_USB:USB_C_Receptacle_GCT_USB4110
- R1: footprint (none) -> Resistor_SMD:R_0805_2012Metric
- R2, R3, R4, R5: footprint (none) -> Resistor_SMD:R_0402_1005Metric
- U2: renamed from U1; footprint DRV6_1X1P6_TEX -> TPS25200:DRV6_1X1P6_TEX
Connections:
- net GND: now also U1.2 (GND)
- net MCU/D+: now also U1.4 (I/O2); no longer J1.A6 (D+), J1.B6 (D+)
- net MCU/D-: now also U1.6 (I/O1); no longer J1.A7 (D-), J1.B7 (D-)
- net at C2.1, J1.A4 (VBUS), J1.A9 (VBUS)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: now also U1.5 (VBUS)
- new net: J1.A7 (D-), J1.B7 (D-), U1.1 (I/O1)
- new net: J1.A6 (D+), J1.B6 (D+), U1.3 (I/O2)
- no-connect marks 0 -> 1
